File: Hardware/TeensyDrone/TeensyDrone.kicad_sch (KiCad schematic)
At the start: 20 parts, among them J1 Conn_01x04, J2 Conn_01x08, J3 Conn_01x04, U1 DEV-15583

Commit message: Second iteration of PCB
Signed-off-by: lucas <mtglucas1@gmail.com>
Connections:
- net at J3.1 (RX): now also U1.20; no longer U1.14
- net at J3.2 (TX): now also U1.21; no longer U1.15
- net at U1.16: now also J1.3 (GND)
- net at U1.17: now also J1.4 (3.3V)
- net at U1.18: no longer J1.4 (Pin_4)
- net at U1.19: no longer J1.3 (Pin_3)
Changed lines of the file:
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@@
 	)
 	(no_connect
-		(at 171.45 96.52)
+		(at 171.45 99.06)
 	)
 	(no_connect
@@
 	)
 	(no_connect
-		(at 171.45 83.82)
-	)
-	(no_connect
 		(at 57.15 45.72)
 	)
@@
 	)
 	(no_connect
-		(at 171.45 86.36)
-	)
-	(no_connect
 		(at 121.92 58.42)
 	)
@@
 	)
 	(no_connect
-		(at 171.45 93.98)
-	)
-	(no_connect
 		(at 87.63 78.74)
 	)
 	(no_connect
+		(at 171.45 101.6)
+	)
+	(no_connect
+		(at 171.45 88.9)
+	)
+	(no_connect
 		(at 171.45 81.28)
 	)
 	(no_connect
+		(at 171.45 91.44)
+	)
+	(no_connect
 		(at 135.89 111.76)
 	)
@@
 	(wire
 		(pts
-			(xy 176.53 88.9) (xy 176.53 132.08)
-		)
-		(stroke
-			(width 0)
-			(type default)
-		)
-	)
-	(wire
-		(pts
 			(xy 121.92 63.5) (xy 130.81 63.5)
 		)
@@
 	(wire
 		(pts
+			(xy 171.45 96.52) (xy 176.53 96.52)
+		)
+		(stroke
+			(width 0)
+			(type default)
+		)
+	)
+	(wire
+		(pts
 			(xy 185.42 148.59) (xy 121.92 148.59)
 		)
@@
 	(wire
 		(pts
+			(xy 177.8 83.82) (xy 171.45 83.82)
+		)
+		(stroke
+			(width 0)
+			(type default)
+		)
+	)
+	(wire
+		(pts
 			(xy 87.63 144.78) (xy 91.44 144.78)
 		)
@@
 	(wire
 		(pts
+			(xy 177.8 83.82) (xy 177.8 151.13)
+		)
+		(stroke
+			(width 0)
+			(type default)
+		)
+	)
+	(wire
+		(pts
 			(xy 78.74 135.89) (xy 78.74 133.35)
 		)
@@
 	(wire
 		(pts
-			(xy 177.8 99.06) (xy 177.8 151.13)
-		)
-		(stroke
-			(width 0)
-			(type default)
-		)
-	)
-	(wire
-		(pts
 			(xy 124.46 144.78) (xy 181.61 144.78)
 		)
@@
 	(wire
 		(pts
-			(xy 179.07 91.44) (xy 179.07 142.24)
-		)
-		(stroke
-			(width 0)
-			(type default)
-		)
-	)
-	(wire
-		(pts
 			(xy 114.3 156.21) (xy 189.23 156.21)
 		)
@@
 	(wire
 		(pts
-			(xy 171.45 99.06) (xy 177.8 99.06)
-		)
-		(stroke
-			(width 0)
-			(type default)
-		)
-	)
-	(wire
-		(pts
 			(xy 129.54 66.04) (xy 129.54 93.98)
 		)
@@
 	(wire
 		(pts
+			(xy 171.45 93.98) (xy 179.07 93.98)
+		)
+		(stroke
+			(width 0)
+			(type default)
+		)
+	)
+	(wire
+		(pts
 			(xy 114.3 35.56) (xy 179.07 35.56)
 		)
@@
 	(wire
 		(pts
+			(xy 179.07 93.98) (xy 179.07 142.24)
+		)
+		(stroke
+			(width 0)
+			(type default)
+		)
+	)
+	(wire
+		(pts
 			(xy 109.22 153.67) (xy 175.26 153.67)
 		)
@@
 	(wire
 		(pts
+			(xy 175.26 86.36) (xy 175.26 153.67)
+		)
+		(stroke
+			(width 0)
+			(type default)
+		)
+	)
+	(wire
+		(pts
 			(xy 105.41 93.98) (xy 125.73 93.98)
 		)
@@
 	(wire
 		(pts
-			(xy 175.26 101.6) (xy 175.26 153.67)
-		)
-		(stroke
-			(width 0)
-			(type default)
-		)
-	)
-	(wire
-		(pts
 			(xy 85.09 49.53) (xy 85.09 34.29)
 		)
@@
 	(wire
 		(pts
-			(xy 176.53 88.9) (xy 171.45 88.9)
-		)
-		(stroke
-			(width 0)
-			(type default)
-		)
-	)
-	(wire
-		(pts
 			(xy 127 91.44) (xy 127 76.2)
 		)
@@
 	(wire
 		(pts
+			(xy 176.53 96.52) (xy 176.53 132.08)
+		)
+		(stroke
+			(width 0)
+			(type default)
+		)
+	)
+	(wire
+		(pts
+			(xy 175.26 86.36) (xy 171.45 86.36)
+		)
+		(stroke
+			(width 0)
+			(type default)
+		)
+	)
+	(wire
+		(pts
 			(xy 105.41 91.44) (xy 127 91.44)
 		)
@@
 	(wire
 		(pts
-			(xy 171.45 101.6) (xy 175.26 101.6)
-		)
-		(stroke
-			(width 0)
-			(type default)
-		)
-	)
-	(wire
-		(pts
 			(xy 92.71 147.32) (xy 92.71 146.05)
 		)
@@
 		)
 		(stroke
-			(width 0)
-			(type default)
-		)
-	)
-	(wire
-		(pts
-			(xy 171.45 91.44) (xy 179.07 91.44)
-		)
-		(stroke
