File: Hardware/TeensyDrone/TeensyDrone.kicad_sch (KiCad schematic)
At the start: 20 parts, among them J1 Conn_01x04, J2 Conn_01x08, J3 Conn_01x04, U1 DEV-15583

Commit message: Done Hardware Section
Signed-off-by: lucas <mtglucas1@gmail.com>
Parts:
- removed H4: MountingHole, MountingHole:MountingHole_2mm, symbol Mechanical:MountingHole
- added C1: 330 uF, symbol Device:C
- added J4: Conn_01x04, Connector_PinHeader_2.54mm:PinHeader_1x04_P2.54mm_Vertical, symbol Connector_Generic:Conn_01x04
Connections:
- net at U1.20: no longer J3.1 (RX)
- net at U1.21: no longer J3.2 (TX)
- net GND: now reaches 5V_BEC1.5 (GND), J3.3 (GND), U1.G3 (GND), U2.1 (GND)
- net GND: now also 5V_BEC1.1 (GND), ACC1.GND, J1.3 (SCL), J2.1 (Pin_1), U1.G1 (GND), U1.G2 (GND), J4.4 (SDA); no longer J1.2 (SCL), U4.GND
- net 5V: now reaches 5V_BEC1.7 (5V), J3.4 (5V), U1.VIN, U2.2 (VCC), U4.5V
- net 5V: now also J4.3 (SCL)
- net at U1.0: no longer U2.3 (TX)
- net at U1.1: now also J2.6 (Pin_6); no longer U2.4 (RX)
- net ELRS_RX: now reaches U1.14
- net ELRS_RX: now also U2.4 (RX), J4.1 (3.3V)
- net ELRS_TX: now reaches U1.15
- net ELRS_TX: now also U2.3 (TX), J4.2 (GND)
- net OF_TX: now reaches U1.16
- net OF_TX: now also J3.2 (TX); no longer J1.3 (GND)
- net +3.3V: now reaches J1.4 (SDA)
- net +3.3V: now also ACC1.3.3V, U1.3.3V (3.3); no longer U1.17
- net IMU_SDA: now reaches U1.18
- net IMU_SDA: now also ACC1.SDA, J1.1 (3.3V)
- net IMU_SCL: now reaches U1.19
- net IMU_SCL: now also ACC1.SCL, J1.2 (GND)
- net at U1.2: now also J2.5 (Pin_5)
- net at U1.3: now also J2.4 (Pin_4)
- net at U1.4: now also J2.3 (Pin_3)
- net at U1.6: no longer J2.6 (Pin_6)
- net at U1.7: no longer J2.5 (Pin_5)
- net at U1.8: no longer J2.4 (Pin_4)
- net at U1.9: no longer J2.3 (Pin_3)
- net at BT1.1 (+), U3.1 (VCC): now also C1.1
- net at BT1.2 (-), U3.2 (GND): now also C1.2
- net VBat: now reaches 5V_BEC1.3 (VBat), J2.2 (Pin_2)
- new net OF_RX: J3.1 (RX), U1.17
- no-connect marks 44 -> 42
Other:
- note added: "Connections from Mounted Components to the board, which are then routed to the circuit board traces"
- note added: "ESC cannot regulate down to 5V so we need external connection"
- note added: "Peripherals + Serial Communication: ELRS Receiver : UART IMU : I2C (Addr - 0x34) Optical Flow : UART"
- note removed: "Connections from Mounted Components so the board, which are then routed to the circuit board traces ESC:"
- note removed: "Don't fill out traces from IMU to connectors, those will be regular wires in "free space""
- note removed: "There are only 12 Connections to the MC, so most of the components will have X's marking no connection"
- moved on the sheet: 5V_BEC1, ACC1, BT1, H1, H11, H2, H3, H5, H6, H7, H8, H9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
