Commit message: Acquired Hardware In the Loop (HIL)
Signed-off-by: Lucas Wendland <mtglucas1@gmail.com>

File: f_drone_simulation/models/f_drone/model.urdf (robot description, URDF)
Before this commit: robot drone, 5 links, 4 joints
Links:
- removed link propeller
- removed link propeller_2
- removed link propeller_3
- removed link propeller_4
- added link drone_frame, mass 0.152078; collision mesh filename=package://f_drone_simulation/models/f_drone/assets/2s_batte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; collision mesh filename=package://f_drone_simulation/models/f_drone/assets/back_win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
- added link prop, mass 0.000758683; collision mesh filename=package://f_drone_simulation/models/f_drone/assets/prop.stl; visual mesh filename=package://f_drone_simulation/models/f_drone/assets/prop.stl
- added link prop_2, mass 0.000758683; collision mesh filename=package://f_drone_simulation/models/f_drone/assets/prop.stl; visual mesh filename=package://f_drone_simulation/models/f_drone/assets/prop.stl
- added link prop_3, mass 0.000758683; collision mesh filename=package://f_drone_simulation/models/f_drone/assets/prop.stl; visual mesh filename=package://f_drone_simulation/models/f_drone/assets/prop.stl
- added link prop_4, mass 0.000758683; collision mesh filename=package://f_drone_simulation/models/f_drone/assets/prop.stl; visual mesh filename=package://f_drone_simulation/models/f_drone/assets/prop.stl
- link base_link: mass 0.00992449 -> 1e-9; geometry 
Joints:
- added joint base_link_frame: type fixed, parent drone_frame, child base_link, origin xyz=4.27546e-19 1.50726e-19 0.04857 rpy=1.98523e-23 -2.79915e-17 5.69408e-19, axis 0 0 0
- joint motor_prop_1: child propeller_2 -> prop; origin xyz=0.0421043 0.0430423 0.00247314 rpy=3.14159 -0 0 -> xyz=-0.042 -0.0442159 0.057625 rpy=8.78666e-17 -6.99788e-17 3.69828e-18; parent base_link -> drone_frame
- joint motor_prop_2: child propeller -> prop_2; origin xyz=0.0421043 -0.0449577 0.00247314 rpy=3.14159 -0 0 -> xyz=-0.042 0.0437841 0.057625 rpy=3.01379e-17 -4.19873e-17 1.61237e-18; parent base_link -> drone_frame
- joint motor_prop_3: child propeller_3 -> prop_3; origin xyz=-0.0418957 0.0430423 0.00247314 rpy=3.14159 -7.94093e-23 1.42203e-07 -> xyz=0.042 -0.0442159 0.057625 rpy=3.07747e-17 -4.19873e-17 1.78931e-16; parent base_link -> drone_frame
- joint motor_prop_4: child propeller_4 -> prop_4; origin xyz=-0.0418957 -0.0449577 0.00247314 rpy=3.14159 -0 0 -> xyz=0.042 0.0437841 0.057625 rpy=3.07747e-17 -4.19873e-17 1.78931e-16; parent base_link -> drone_frame
